Commit message: Add calibrated follower driver and MoveIt configs

File: nakalab_so101_description/urdf/_so101.urdf.xacro (robot description, xacro)
@@ -409,75 +409,4 @@
       <limit effort="10" velocity="10" lower="-1.91986" upper="1.91986"/>
     </joint>
-    <ros2_control name="NGSRHardware" type="system">
-      <hardware>
-        <plugin>ngsr_controller/NGSRHardware</plugin>
-      </hardware>
-      <joint name="shoulder_pan">
-        <command_interface name="position">
-          <param name="min">-1.91986</param>
-          <param name="max">1.91986</param>
-        </command_interface>
-        <state_interface name="position">
-          <param name="initial_value">0.0</param>
-        </state_interface>
-        <state_interface name="velocity"/>
-        <state_interface name="effort"/>
-      </joint>
-      <joint name="shoulder_lift">
-        <command_interface name="position">
-          <param name="min">-1.74533</param>
-          <param name="max">1.74533</param>
-        </command_interface>
-        <state_interface name="position">
-          <param name="initial_value">0.0</param>
-        </state_interface>
-        <state_interface name="velocity"/>
-        <state_interface name="effort"/>
-      </joint>
-      <joint name="elbow_flex">
-        <command_interface name="position">
-          <param name="min">-1.69</param>
-          <param name="max">1.69</param>
-        </command_interface>
-        <state_interface name="position">
-          <param name="initial_value">0.0</param>
-        </state_interface>
-        <state_interface name="velocity"/>
-        <state_interface name="effort"/>
-      </joint>
-      <joint name="wrist_flex">
-        <command_interface name="position">
-          <param name="min">-1.65806</param>
-          <param name="max">1.65806</param>
-        </command_interface>
-        <state_interface name="position">
-          <param name="initial_value">0.0</param>
-        </state_interface>
-        <state_interface name="velocity"/>
-        <state_interface name="effort"/>
-      </joint>
-      <joint name="wrist_roll">
-        <command_interface name="position">
-          <param name="min">-2.74385</param>
-          <param name="max">2.84121</param>
-        </command_interface>
-        <state_interface name="position">
-          <param name="initial_value">0.0</param>
-        </state_interface>
-        <state_interface name="velocity"/>
-        <state_interface name="effort"/>
-      </joint>
-      <joint name="gripper">
-        <command_interface name="position">
-          <param name="min">-0.174533</param>
-          <param name="max">1.74533</param>
-        </command_interface>
-        <state_interface name="position">
-          <param name="initial_value">0.0</param>
-        </state_interface>
-        <state_interface name="velocity"/>
-        <state_interface name="effort"/>
-      </joint>
-    </ros2_control>
   </xacro:macro>
 </robot>

Commit message: Dupdate

File: nakalab_so101_description/urdf/_so101.urdf.xacro (robot description, xacro)
@@ -331,6 +331,6 @@
     <xacro:if value="${camera_type == 'd435'}">
         <xacro:include filename="$(find nakalab_realsense)/urdf/_d435.urdf.xacro" />
-        <xacro:sensor_d435 parent="d435_mounter_link" name="so101_camera" use_nominal_extrinsics="true">
-            <origin xyz="0.005 0.0025 0.017" rpy="3.14159 2.75 0.04"/>
+        <xacro:sensor_d435 parent="d435_mounter_link" name="so101_camera" use_nominal_extrinsics="false">
+            <origin xyz="0.005 0.011 0.017" rpy="3.14159 2.725 0.04"/>
         </xacro:sensor_d435>
         <link name="d435_mounter_link">
